File: FIRM.kicad_sch (KiCad schematic)
At the start: 80 parts, among them J1 DM3CS-SF, J2 Conn_01x02_Pin, Q1 IRLML6402, U1 W25Q128JVS, U2 STM32F405RGTx, U3 ADXL371, U5 INA219AxDCN, U6 MIC5219-3.3YM5, U9 A-USBC-20F0-EA-GSR05, X1 32.768khz, Y1 12 MHz

Commit message: new stm and flash
Parts:
- removed C12: 100n, Capacitor_SMD:C_0402_1005Metric, symbol Device:C_Small
- removed C4, C7: 6p, Capacitor_SMD:C_0402_1005Metric, symbol Device:C
- removed J1: DM3CS-SF, connectors:HRS_DM3CS-SF, symbol connectors:DM3CS-SF
- removed R1, R2, R4, R5, R6, R7: 47k, Resistor_SMD:R_0402_1005Metric, symbol Device:R_Small
- removed RN2: 10k, connectors:R_Array_YC104, symbol Device:R_Pack04
- removed U1: W25Q128JVS, Package_SO:SOIC-8_5.3x5.3mm_P1.27mm, symbol Memory_Flash:W25Q128JVS
- removed U2: STM32F405RGTx, Package_QFP:LQFP-64_10x10mm_P0.5mm, symbol MCU_ST_STM32F4:STM32F405RGTx
- removed X1: 32.768khz, connectors:Crystal_ECS-.327-6-12RR-TR, symbol Device:Crystal
- added R1: 10k, Resistor_SMD:R_0402_1005Metric, symbol Device:R
- added U1: W25N04KVZEIR, IC_W25N04KVZEIR:IC_W25N04KVZEIR, symbol W25N04KVZEIR:W25N04KVZEIR
- added U2: STM32H743VIHx, Package_BGA:TFBGA-100_8x8mm_Layout10x10_P0.8mm, symbol MCU_ST_STM32H7:STM32H743VIHx
- C1: Digikey PN 1276-1043-1-ND -> 1276-1482-1-ND; MPN C1590 -> C1705
- C10, C5: value 14p -> 10p
- R13: value 330 -> 1.2k
- R15: value 1k5 -> 1k2
- R3: value 100k -> 10k
- Y1: value 12 MHz -> 25 MHz; footprint connectors:Crystal_ECS-120-10-36B2-CWY-TR -> Crystal:Crystal_SMD_3225-4Pin_3.2x2.5mm; Digikey PN 50-ECS-120-10-36B2-CWY-TRCT-ND -> 644-STDCRG2-25MCT-ND
Connections:
- net +3.3V: now also R1.2, U1.8 (VCC), U2.B2 (VBAT), U2.D2 (VDD), U2.F5 (VDD), U2.F6 (VDD33_USB), U2.F7 (PDR_ON), U2.K1 (VDD)
- net GND: now also U1.4 (GND), U1.9 (EXP)
- net I2C1_SCL: no longer R11.1
- net I2C1_SDA: no longer R12.1
- net SWCLK: no longer TP13.1
- net at C16.1, C17.1, FB1.1: now also U2.H1 (VDDA)
- net BOOT0: no longer names the net of R3.1
- net BOOT0: now also U2.D5 (BOOT0)
- net HSE_IN: no longer names the net of C5.1, Y1.1
- net HSE_IN: now also U2.C1 (PH0)
- net HSE_OUT: no longer names the net of C10.1, Y1.3
- net HSE_OUT: now also U2.D1 (PH1)
- net NRST: no longer names the net of C1.1, TP24.1
- net NRST: now also U2.E1 (NRST)
- net SWDIO: no longer names the net of TP12.1
- net VCAP1: no longer names the net of C9.1
- net VCAP1: now also U2.E7 (VCAP)
- net VCAP2: no longer names the net of C14.1
- net VCAP2: now also U2.F8 (VCAP)
- new net: R1.1, U1.1 (~{CS})
- new net: U2.C2 (VSS), U2.E4 (VSS), U2.E5 (VSS), U2.E6 (VSS), U2.J1 (VSS)
- new net: U3.10 (RES), U3.13 (GND), U3.16 (GND)
- no-connect marks 21 -> 20
Other:
- moved on the sheet: C10, C14, C5, C9, R11, R3, TP1, TP14, TP2, TP24, TP3, TP4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

Commit message: Update FIRM.kicad_sch
Started updating STM32H743VITx schematic
Parts:
- added C12, C31, C32, C33, C35, C39, C7: 100n, Capacitor_SMD:C_0402_1005Metric, symbol Device:C
- added C34, C36, C40: 1u, Capacitor_SMD:C_0402_1005Metric, symbol Device:C
- added C37, C38: 2u2, Capacitor_SMD:C_0402_1005Metric, symbol Device:C
- added C4: 4u7, Capacitor_SMD:C_0402_1005Metric, symbol Device:C
- added FB2: 120 Ohms @ 100 MHz, Inductor_SMD:L_0603_1608Metric, symbol Device:FerriteBead
- added U10: STM32H743VITx, Package_QFP:LQFP-100_14x14mm_P0.5mm, symbol MCU_ST_STM32H7:STM32H743VITx
Connections:
- net +3.3V: now also C12.1, C31.1, C32.1, C33.1, C36.1, C4.1, C7.1, FB2.2, U10.100 (VDD), U10.11 (VDD), U10.27 (VDD), U10.50 (VDD), U10.6 (VBAT), U10.75 (VDD)
- net GND: now also C12.2, C31.2, C32.2, C33.2, C34.2, C35.2, C36.2, C37.2, C38.2, C39.2, C4.2, C40.2, C7.2, U10.10 (VSS), U10.26 (VSS), U10.49 (VSS), U10.74 (VSS), U10.99 (VSS)
- new net: C39.1, C40.1, U10.20 (VREF+)
- new net: C34.1, C35.1, FB2.1, U10.21 (VDDA)
- new net: C37.1, U10.48 (VCAP)
- new net: C38.1, U10.73 (VCAP)
- new net: U3.10 (RES), U3.13 (GND), U3.16 (GND)
Other:
- moved on the sheet: C1, C10, C13, C14, C15, C16, C17, C18, C2, C3, C5, C6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

Commit message: Update FIRM.kicad_sch
Connections:
- net GND: no longer U10.10 (VSS), U10.26 (VSS), U10.49 (VSS), U10.74 (VSS), U10.99 (VSS)
- new net: U10.10 (VSS), U10.26 (VSS), U10.49 (VSS), U10.74 (VSS), U10.99 (VSS)
- new net: U3.10 (RES), U3.13 (GND), U3.16 (GND)
Changed lines of the file:
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@@
-	)
-	(symbol
-		(lib_id "power:GND")
-		(at 102.87 184.15 0)
-		(unit 1)
-		(exclude_from_sim no)
-		(in_bom yes)
-		(on_board yes)
-		(dnp no)
-		(property "Reference" "#PWR015"
-			(at 102.87 190.5 0)
-			(effects
-				(font
-					(size 1.27 1.27)
-				)
-				(hide yes)
-			)
-		)
-		(property "Value" "GND"
-			(at 102.87 187.706 0)
-			(effects
-				(font
-					(size 1.27 1.27)
-				)
-			)
-		)
-		(property "Footprint" ""
-			(at 102.87 184.15 0)
-			(effects
-				(font
-					(size 1.27 1.27)
-				)
-				(hide yes)
-			)
-		)
-		(property "Datasheet" ""
-			(at 102.87 184.15 0)
-			(effects
-				(font
-					(size 1.27 1.27)
-				)
-				(hide yes)
-			)
-		)
-		(property "Description" "Power symbol creates a global label with name \"GND\" , ground"
-			(at 102.87 184.15 0)
-			(effects
-				(font
-					(size 1.27 1.27)
-				)
-				(hide yes)
-			)
-		)
-		(pin "1"
-		)
-		(instances
-			(project "FIRM"
-				(path "/d3f8a00a-ef65-439d-87f3-373a106a7ddb"
-					(reference "#PWR015")
-					(unit 1)
-				)
-			)
-		)
 	)
 	(symbol
