File: FIRM v1.1/FIRM.kicad_sch (KiCad schematic)
At the start: 116 parts, among them J2 Conn_01x02_Pin, Q1 IRLML6402, U1 W25N04KVZEIR, U10 STM32F446ZCHx, U2 STM32H743VIHx, U3 ADXL371, U5 INA219AxDCN, U6 MIC5219-3.3YM5, U9 A-USBC-20F0-EA-GSR05, Y1 25 MHz, Y2 12 MHz

Commit message: Save in KiCad 10.0
Parts:
- U4, U7, U8: value ~ -> (none)
Connections:
- new net: U3.10 (RES), U3.13 (GND), U3.16 (GND)
