File: FIRM v1.1/FIRM_v1.1.kicad_sch (KiCad schematic)
At the start: 94 parts, among them J1 Pin, J2 Conn_01x02_Pin, J3 FIRM2 Conn, Q2 DMP3098L-7, U11 SCH16T-K01-10, U12 STM32F446ZCHx, U5 INA219AxDCN, U9 A-USBC-20F0-EA-GSR05, Y1 12 MHz

Commit message: Wired the TPS2121 and added USB sensing to STM
I have implemented the TPS2121 into the power circuit. I gave N1 priority, switching if Vbus falls bellow 4.25. I gave IN2 a Overvoltage value of 15. limited the current to two amps,  and set up the TPS2121 to protect agains polirazation. Added a bulk capacitor to account for switching time at OUT and two ceramics in INs.
Parts:
- removed D4: D_Schottky, HPRC_Connectors:D_schottky_NSR05F30NXT5G, symbol Device:D_Schottky
- removed Q2: DMP3098L-7, HPRC_Logic:DMP3098L-7, symbol HPRC_Logic_ICs:DMP3098L-7
- removed R16: 100k, Resistor_SMD:R_0402_1005Metric, symbol Device:R
- added C28: 10u, Capacitor_SMD:C_0603_1608Metric, symbol Device:C_Small
- added C32: 10u, Capacitor_SMD:C_0805_2012Metric, symbol Device:C_Small
- added C5: 100u, Capacitor_SMD:CP_Elec_8x5.4, symbol Device:C
- added C60: 1u, Capacitor_SMD:C_0402_1005Metric, symbol Device:C
- added D6: D_Schottky, HPRC_Connectors:D_schottky_NSR05F30NXT5G, symbol Device:D_Schottky
- added R27, R30: 100k, Resistor_SMD:R_0402_1005Metric, symbol Device:R_Small
- added R28: 301k, Resistor_SMD:R_0402_1005Metric, symbol Device:R_Small
- added R29: 1.3M, Resistor_SMD:R_0402_1005Metric, symbol Device:R_Small
- added R31: 57.6k, Resistor_SMD:R_0402_1005Metric, symbol Device:R_Small
- added R35: 5.1k, Resistor_SMD:R_0402_1005Metric, symbol Device:R_Small
- added R36: 10k, Resistor_SMD:R_0402_1005Metric, symbol Device:R_Small
- added U3: TPS2121RUXR, HPRC_Regulators:IC_TPS2121RUXR, symbol HPRC_Regulators:TPS2121RUXR
- C26, C31: footprint Capacitor_SMD:C_0603_1608Metric -> Capacitor_SMD:C_0805_2012Metric
Connections:
- net GND: now also C28.2, C32.1, C5.2, D6.1 (K), R36.2
- net VBAT: now also C32.2, R29.1, U3.2 (IN2), U3.2_1 (IN2)
- net VBUS: now also C28.1, R28.1, R35.1, U3.7 (IN1), U3.7_1 (IN1)
- net VSENS_IN: now also C5.1, U3.1 (OUT), U3.1_1 (OUT), U3.8 (OUT), U3.8_1 (OUT)
- net USB_SENS: now reaches U12.D12 (PA9)
- net USB_SENS: now also R35.2, R36.1
- new net: R27.1, R28.2, U3.6 (PR1)
- new net: R29.2, R30.1, U3.4 (OV2)
- new net: C60.1, U3.11 (SS)
- new net: R31.1, U3.10 (ILIM)
- new net GND_Device: C60.2, D6.2 (A), R27.2, R30.2, R31.2, U3.12 (GND), U3.3 (CP2), U3.5 (OV1), U3.9 (ST)
- no-connect marks 95 -> 94
Other:
- moved on the sheet: C26, C31, D5, J2, L1, PS1, R18, R20, R21, R26, U9

Commit message: I changed the schematic to enable t_FSW. I made my Vref=2.5 and modified my resistor values so PR1 and OV2 stayed the same.
Parts:
- added R37, R38: 100k, Resistor_SMD:R_0402_1005Metric, symbol Device:R_Small
- R28: value 301k -> 80k
- R29: value 1.3M -> 100k
- R30: value 100k -> 20k
Connections:
- net GND_Device: now also R38.2; no longer U3.3 (CP2)
- net VBUS: now also R37.1
- new net: R37.2, R38.1, U3.3 (CP2)
Other:
- moved on the sheet: R30
Changed lines of the file:
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@@
 	)
 	(junction
+		(at 340.36 218.44)
+		(diameter 0)
+		(color 0 0 0 0)
+	)
+	(junction
 		(at 346.71 233.68)
 		(diameter 0)
@@
 	)
 	(junction
-		(at 344.17 248.92)
-		(diameter 0)
-		(color 0 0 0 0)
-	)
-	(junction
 		(at 107.95 102.87)
 		(diameter 0)
@@
 	)
 	(junction
+		(at 340.36 246.38)
+		(diameter 0)
+		(color 0 0 0 0)
+	)
+	(junction
 		(at 554.99 54.61)
 		(diameter 0)
@@
 	(wire
 		(pts
-			(xy 332.74 218.44) (xy 346.71 218.44)
+			(xy 332.74 218.44) (xy 340.36 218.44)
 		)
 		(stroke
@@
 	(wire
 		(pts
+			(xy 340.36 246.38) (xy 359.41 246.38)
+		)
+		(stroke
+			(width 0)
+			(type default)
+		)
+	)
+	(wire
+		(pts
 			(xy 535.94 36.83) (xy 535.94 39.37)
 		)
@@
 	(wire
 		(pts
+			(xy 340.36 246.38) (xy 340.36 251.46)
+		)
+		(stroke
+			(width 0)
+			(type default)
+		)
+	)
+	(wire
+		(pts
 			(xy 429.26 257.81) (xy 491.49 257.81)
 		)
@@
 	(wire
 		(pts
+			(xy 340.36 227.33) (xy 340.36 218.44)
+		)
+		(stroke
+			(width 0)
+			(type default)
+		)
+	)
+	(wire
+		(pts
+			(xy 340.36 218.44) (xy 346.71 218.44)
+		)
+		(stroke
+			(width 0)
+			(type default)
+		)
+	)
+	(wire
+		(pts
 			(xy 85.09 52.07) (xy 85.09 53.34)
 		)
@@
 	(wire
 		(pts
-			(xy 353.06 248.92) (xy 353.06 246.38)
-		)
-		(stroke
-			(width 0)
-			(type default)
-		)
-	)
-	(wire
-		(pts
 			(xy 49.53 52.07) (xy 49.53 53.34)
 		)
@@
 	(wire
 		(pts
-			(xy 353.06 246.38) (xy 359.41 246.38)
-		)
-		(stroke
-			(width 0)
-			(type default)
-		)
-	)
-	(wire
-		(pts
 			(xy 114.3 186.69) (xy 116.84 186.69)
 		)
@@
 	(wire
 		(pts
+			(xy 340.36 232.41) (xy 340.36 246.38)
+		)
+		(stroke
+			(width 0)
+			(type default)
+		)
+	)
+	(wire
+		(pts
 			(xy 142.24 81.28) (xy 146.05 81.28)
 		)
@@
 	(wire
 		(pts
+			(xy 344.17 250.19) (xy 344.17 243.84)
+		)
+		(stroke
+			(width 0)
+			(type default)
+		)
+	)
+	(wire
+		(pts
 			(xy 452.12 40.64) (xy 452.12 43.18)
 		)
@@
 	(wire
 		(pts
+			(xy 340.36 264.16) (xy 344.17 264.16)
+		)
+		(stroke
+			(width 0)
+			(type default)
+		)
+	)
+	(wire
+		(pts
 			(xy 476.25 243.84) (xy 476.25 257.81)
 		)
@@
 	(wire
 		(pts
-			(xy 344.17 264.16) (xy 344.17 248.92)
+			(xy 344.17 264.16) (xy 344.17 255.27)
 		)
 		(stroke
@@
 	(wire
 		(pts
+			(xy 340.36 256.54) (xy 340.36 264.16)
+		)
+		(stroke
+			(width 0)
+			(type default)
+		)
+	)
+	(wire
+		(pts
 			(xy 154.94 52.07) (xy 154.94 53.34)
 		)
@@
 	(wire
 		(pts
-			(xy 344.17 248.92) (xy 353.06 248.92)
-		)
-		(stroke
-			(width 0)
-			(type default)
-		)
-	)
-	(wire
-		(pts
 			(xy 429.26 226.06) (xy 429.26 236.22)
 		)
@@
 	)
 	(symbol
+		(lib_id "Device:R_Small")
+		(at 340.36 229.87 0)
+		(unit 1)
+		(body_style 1)
+		(exclude_from_sim no)
+		(in_bom yes)
+		(on_board yes)
+		(in_pos_files yes)
+		(dnp no)
+		(property "Reference" "R37"
+			(at 341.376 230.124 0)
+			(show_name no)
+			(do_not_autoplace no)
+			(effects
+				(font
+					(size 1.016 1.016)
+				)
+				(justify left)
+			)
+		)
+		(property "Value" "100k"
+			(at 341.376 232.664 0)
+			(show_name no)
+			(do_not_autoplace no)
+			(effects
+				(font
+					(size 1.27 1.27)
+				)
+				(justify left)
+			)
+		)
+		(property "Footprint" "Resistor_SMD:R_0402_1005Metric"
+			(at 340.36 229.87 0)
+			(hide yes)
+			(show_name no)
+			(do_not_autoplace no)
+			(effects
+				(font
+					(size 1.27 1.27)
+				)
+			)
+		)
+		(property "Datasheet" ""
+			(at 340.36 229.87 0)
+			(hide yes)
+			(show_name no)
+			(do_not_autoplace no)
+			(effects
+				(font
+					(size 1.27 1.27)
+				)
+			)
+		)
+		(property "Description" "Resistor, small symbol"
+			(at 340.36 229.87 0)
+			(hide yes)
+			(show_name no)
+			(do_not_autoplace no)
+			(effects
+				(font
+					(size 1.27 1.27)
+				)
+			)
+		)
+		(pin "1"
+		)
+		(pin "2"
+		)
+		(instances
+			(project "FIRM_v1.1"
+				(path "/d3f8a00a-ef65-439d-87f3-373a106a7ddb"
+					(reference "R37")
+					(unit 1)
+				)
+			)
+		)
+	)
+	(symbol
 		(lib_id "power:GND")
 		(at 125.73 73.66 0)
@@
 	(symbol
 		(lib_id "Device:R_Small")
+		(at 340.36 254 0)
+		(unit 1)
+		(body_style 1)
+		(exclude_from_sim no)
+		(in_bom yes)
+		(on_board yes)
+		(in_pos_files yes)
+		(dnp no)
+		(property "Reference" "R38"
+			(at 334.772 252.984 0)
+			(show_name no)
+			(do_not_autoplace no)
+			(effects
+				(font
+					(size 1.016 1.016)
+				)
+				(justify left)
+			)
+		)
+		(property "Value" "100k"
+			(at 334.772 255.524 0)
+			(show_name no)
+			(do_not_autoplace no)
+			(effects
+				(font
+					(size 1.27 1.27)
+				)
+				(justify left)
+			)
+		)
+		(property "Footprint" "Resistor_SMD:R_0402_1005Metric"
+			(at 340.36 254 0)
+			(hide yes)
+			(show_name no)
+			(do_not_autoplace no)
+			(effects
+				(font
+					(size 1.27 1.27)
+				)
+			)
+		)
+		(property "Datasheet" ""
+			(at 340.36 254 0)
+			(hide yes)
+			(show_name no)
+			(do_not_autoplace no)
+			(effects
+				(font
+					(size 1.27 1.27)
+				)
+			)
+		)
+		(property "Description" "Resistor, small symbol"
+			(at 340.36 254 0)
+			(hide yes)
+			(show_name no)
+			(do_not_autoplace no)
+			(effects
+				(font
+					(size 1.27 1.27)
+				)
+			)
+		)
+		(pin "1"
+		)
+		(pin "2"
+		)
+		(instances
+			(project "FIRM_v1.1"
+				(path "/d3f8a00a-ef65-439d-87f3-373a106a7ddb"
+					(reference "R38")
+					(unit 1)
+				)
+			)
+		)
+	)
+	(symbol
+		(lib_id "Device:R_Small")
 		(at 346.71 220.98 0)
 		(unit 1)
@@
 			)
 		)
-		(property "Value" "301k"
+		(property "Value" "80k"
 			(at 349.25 222.2499 0)
 			(show_name no)
@@
 	(symbol
 		(lib_id "Device:R_Small")
-		(at 344.17 246.38 0)
+		(at 344.17 252.73 0)
 		(unit 1)
 		(body_style 1)
@@
 		(dnp no)
 		(property "Reference" "R30"
-			(at 337.566 245.364 0)
+			(at 345.44 247.65 0)
 			(show_name no)
 			(do_not_autoplace no)
@@
 			)
 		)
-		(property "Value" "100k"
-			(at 337.566 247.904 0)
+		(property "Value" "20k"
+			(at 345.44 250.19 0)
 			(show_name no)
 			(do_not_autoplace no)
@@
 		)
 		(property "Footprint" "Resistor_SMD:R_0402_1005Metric"
-			(at 344.17 246.38 0)
+			(at 344.17 252.73 0)
 			(hide yes)
 			(show_name no)
@@
 		)
 		(property "Datasheet" ""
-			(at 344.17 246.38 0)
+			(at 344.17 252.73 0)
 			(hide yes)
 			(show_name no)
@@
 		)
 		(property "Description" "Resistor, small symbol"
-			(at 344.17 246.38 0)
+			(at 344.17 252.73 0)
 			(hide yes)
 			(show_name no)
@@
 			)
 		)
-		(property "Value" "1.3M"
+		(property "Value" "100k"
 			(at 346.71 242.5699 0)
 			(show_name no)
@@
 		)
 		(property "Value" "GND"
-			(at 338.582 230.378 0)
+			(at 335.026 227.33 0)
 			(show_name no)
 			(do_not_autoplace no)

Commit message: Fixed Resistor dividers
Parts:
- removed C5: 100u, Capacitor_SMD:CP_Elec_8x5.4, symbol Device:C
- R30: value 20k -> 7k6
- R37: value 100k -> 32
Connections:
- net +3.3V: now also R37.1
- net VBUS: no longer R37.1
Other:
- moved on the sheet: R37
Changed lines of the file:
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@@
 	)
 	(junction
-		(at 340.36 218.44)
-		(diameter 0)
-		(color 0 0 0 0)
-	)
-	(junction
 		(at 346.71 233.68)
 		(diameter 0)
@@
 	)
 	(junction
-		(at 397.51 228.6)
-		(diameter 0)
-		(color 0 0 0 0)
-	)
-	(junction
 		(at 285.75 135.89)
 		(diameter 0)
@@
 	(wire
 		(pts
-			(xy 332.74 218.44) (xy 340.36 218.44)
+			(xy 332.74 218.44) (xy 346.71 218.44)
 		)
 		(stroke
@@
 	(wire
 		(pts
-			(xy 340.36 227.33) (xy 340.36 218.44)
-		)
-		(stroke
-			(width 0)
-			(type default)
-		)
-	)
-	(wire
-		(pts
-			(xy 340.36 218.44) (xy 346.71 218.44)
-		)
-		(stroke
-			(width 0)
-			(type default)
-		)
-	)
-	(wire
-		(pts
 			(xy 85.09 52.07) (xy 85.09 53.34)
 		)
@@
 	(wire
 		(pts
+			(xy 323.85 241.3) (xy 340.36 241.3)
+		)
+		(stroke
+			(width 0)
+			(type default)
+		)
+	)
+	(wire
+		(pts
 			(xy 107.95 88.9) (xy 185.42 88.9)
 		)
@@
 	(wire
 		(pts
-			(xy 397.51 228.6) (xy 398.78 228.6)
+			(xy 384.81 228.6) (xy 398.78 228.6)
 		)
 		(stroke
@@
 	(wire
 		(pts
-			(xy 340.36 232.41) (xy 340.36 246.38)
-		)
-		(stroke
-			(width 0)
-			(type default)
-		)
-	)
-	(wire
-		(pts
 			(xy 142.24 81.28) (xy 146.05 81.28)
 		)
@@
 	(wire
 		(pts
-			(xy 384.81 228.6) (xy 397.51 228.6)
-		)
-		(stroke
-			(width 0)
-			(type default)
-		)
-	)
-	(wire
-		(pts
 			(xy 185.42 154.94) (xy 180.34 154.94)
 		)
@@
 	(symbol
 		(lib_id "Device:R_Small")
-		(at 340.36 229.87 0)
+		(at 340.36 243.84 0)
 		(unit 1)
 		(body_style 1)
@@
 		(dnp no)
 		(property "Reference" "R37"
-			(at 341.376 230.124 0)
+			(at 336.042 242.824 0)
 			(show_name no)
 			(do_not_autoplace no)
@@
 			)
 		)
-		(property "Value" "100k"
-			(at 341.376 232.664 0)
+		(property "Value" "32"
+			(at 336.042 245.364 0)
 			(show_name no)
 			(do_not_autoplace no)
@@
 		)
 		(property "Footprint" "Resistor_SMD:R_0402_1005Metric"
-			(at 340.36 229.87 0)
+			(at 340.36 243.84 0)
 			(hide yes)
 			(show_name no)
@@
 		)
 		(property "Datasheet" ""
-			(at 340.36 229.87 0)
+			(at 340.36 243.84 0)
 			(hide yes)
 			(show_name no)
@@
 		)
 		(property "Description" "Resistor, small symbol"
-			(at 340.36 229.87 0)
+			(at 340.36 243.84 0)
 			(hide yes)
 			(show_name no)
@@
 	(symbol
 		(lib_id "power:GND")
-		(at 397.51 236.22 0)
-		(unit 1)
-		(body_style 1)
-		(exclude_from_sim no)
-		(in_bom yes)
-		(on_board yes)
-		(in_pos_files yes)
-		(dnp no)
-		(property "Reference" "#PWR063"
-			(at 397.51 242.57 0)
-			(hide yes)
-			(show_name no)
-			(do_not_autoplace no)
-			(effects
-				(font
-					(size 1.27 1.27)
-				)
-			)
-		)
-		(property "Value" "GND"
-			(at 400.812 237.998 0)
-			(show_name no)
-			(do_not_autoplace no)
-			(effects
-				(font
-					(size 1.27 1.27)
-				)
-			)
-		)
-		(property "Footprint" ""
-			(at 397.51 236.22 0)
-			(hide yes)
-			(show_name no)
-			(do_not_autoplace no)
-			(effects
-				(font
-					(size 1.27 1.27)
-				)
-			)
-		)
-		(property "Datasheet" ""
-			(at 397.51 236.22 0)
-			(hide yes)
-			(show_name no)
-			(do_not_autoplace no)
-			(effects
-				(font
-					(size 1.27 1.27)
-				)
-			)
-		)
-		(property "Description" "Power symbol creates a global label with name \"GND\" , ground"
-			(at 397.51 236.22 0)
-			(hide yes)
-			(show_name no)
-			(do_not_autoplace no)
-			(effects
-				(font
-					(size 1.27 1.27)
-				)
-			)
-		)
-		(pin "1"
-		)
-		(instances
-			(project "FIRM_v1.1"
-				(path "/d3f8a00a-ef65-439d-87f3-373a106a7ddb"
-					(reference "#PWR063")
-					(unit 1)
-				)
-			)
-		)
-	)
-	(symbol
-		(lib_id "power:GND")
 		(at 490.22 64.77 0)
 		(unit 1)
@@
 			)
 		)
-		(property "Value" "20k"
+		(property "Value" "7k6"
 			(at 345.44 250.19 0)
 			(show_name no)
@@
 	)
 	(symbol
+		(lib_id "power:+3.3V")
+		(at 323.85 241.3 0)
+		(unit 1)
+		(body_style 1)
+		(exclude_from_sim no)
+		(in_bom yes)
+		(on_board yes)
+		(in_pos_files yes)
+		(dnp no)
+		(property "Reference" "#PWR066"
+			(at 323.85 245.11 0)
+			(hide yes)
+			(show_name no)
+			(do_not_autoplace no)
+			(effects
+				(font
+					(size 1.27 1.27)
+				)
+			)
+		)
+		(property "Value" "+3.3V"
+			(at 320.548 237.998 0)
+			(show_name no)
+			(do_not_autoplace no)
+			(effects
+				(font
+					(size 1.27 1.27)
+				)
+			)
+		)
+		(property "Footprint" ""
+			(at 323.85 241.3 0)
+			(hide yes)
+			(show_name no)
+			(do_not_autoplace no)
+			(effects
+				(font
+					(size 1.27 1.27)
+				)
+			)
+		)
+		(property "Datasheet" ""
+			(at 323.85 241.3 0)
+			(hide yes)
+			(show_name no)
+			(do_not_autoplace no)
+			(effects
+				(font
+					(size 1.27 1.27)
+				)
+			)
+		)
+		(property "Description" "Power symbol creates a global label with name \"+3.3V\""
+			(at 323.85 241.3 0)
+			(hide yes)
+			(show_name no)
+			(do_not_autoplace no)
+			(effects
+				(font
+					(size 1.27 1.27)
+				)
+			)
+		)
+		(pin "1"
+		)
+		(instances
+			(project "FIRM_v1.1"
+				(path "/d3f8a00a-ef65-439d-87f3-373a106a7ddb"
+					(reference "#PWR066")
+					(unit 1)
+				)
+			)
+		)
+	)
+	(symbol
 		(lib_id "Device:L_Small")
 		(at 472.44 226.06 90)
@@
 					(unit 1)
 				)
-			)
-		)
-	)
-	(symbol
-		(lib_id "Device:C")
-		(at 397.51 232.41 0)
-		(unit 1)
-		(body_style 1)
-		(exclude_from_sim no)
-		(in_bom yes)
-		(on_board yes)
-		(in_pos_files yes)
-		(dnp no)
-		(property "Reference" "C5"
-			(at 401.32 231.1399 0)
-			(show_name no)
-			(do_not_autoplace no)
-			(effects
-				(font
-					(size 1.27 1.27)
-				)
-				(justify left)
-			)
-		)
-		(property "Value" "100u"
-			(at 401.32 233.6799 0)
-			(show_name no)
-			(do_not_autoplace no)
-			(effects
-				(font
-					(size 1.27 1.27)
-				)
-				(justify left)
-			)
-		)
-		(property "Footprint" "Capacitor_SMD:CP_Elec_8x5.4"
-			(at 398.4752 236.22 0)
-			(hide yes)
-			(show_name no)
-			(do_not_autoplace no)
-			(effects
-				(font
-					(size 1.27 1.27)
-				)
-			)
-		)
-		(property "Datasheet" "https://www.nichicon.co.jp/english/series_items/catalog_pdf/e-pcm.pdf"
-			(at 397.51 232.41 0)
-			(hide yes)
-			(show_name no)
-			(do_not_autoplace no)
-			(effects
-				(font
-					(size 1.27 1.27)
-				)
-			)
-		)
-		(property "Description" "Unpolarized capacitor"
-			(at 397.51 232.41 0)
-			(hide yes)
-			(show_name no)
-			(do_not_autoplace no)
-			(effects
-				(font
-					(size 1.27 1.27)
-				)
-			)
-		)
-		(property "MPN" "C1705"
-			(at 397.51 232.41 0)
-			(hide yes)
-			(show_name no)
-			(do_not_autoplace no)
-			(effects
-				(font
-					(size 1.27 1.27)
-				)
-			)
-		)
-		(property "Digikey PN" "1276-1482-1-ND"
-			(at 397.51 232.41 0)
-			(hide yes)
-			(show_name no)
-			(do_not_autoplace no)
-			(effects
-				(font
-					(size 1.27 1.27)
-				)
-			)
-		)
-		(pin "1"
-		)
-		(pin "2"
-		)
-		(instances
-			(project "FIRM_v1.1"
-				(path "/d3f8a00a-ef65-439d-87f3-373a106a7ddb"
-					(reference "C5")
-					(unit 1)
-				)

Commit message: fixes
Parts:
- removed C2: 100n, Capacitor_Tantalum_SMD:CP_EIA-1608-08_AVX-J, symbol Device:C_Small
- removed C61, C65: 100n, Capacitor_SMD:C_0402_1005Metric, symbol Device:C_Small
- removed C64: 1u, Capacitor_SMD:C_0402_1005Metric, symbol Device:C_Small
- added C33, C37: 1u, Capacitor_SMD:C_0402_1005Metric, symbol Device:C_Small
- added C35, C36: 100n, Capacitor_SMD:C_0402_1005Metric, symbol Device:C_Small
- added C38: 22u, Capacitor_SMD:C_0805_2012Metric, symbol Device:C_Small
- added R39: 0, Resistor_SMD:R_0201_0603Metric, symbol Device:R_Small
- C26, C32: footprint Capacitor_SMD:C_0805_2012Metric -> Capacitor_SMD:C_0603_1608Metric; Digikey PN 1276-1451-1-ND -> 490-12737-1-ND; MPN C1691 -> GRM188R61E106MA73J
- C28: Digikey PN 1276-1451-1-ND -> 490-12737-1-ND; MPN C1691 -> GRM188R61E106MA73J
- C31: footprint Capacitor_SMD:C_0805_2012Metric -> Capacitor_SMD:C_0603_1608Metric; Digikey PN 1276-1451-1-ND -> 1276-2867-1-ND; MPN C1691 -> CL10A226KQ8NRNE
- C46, C47: Digikey PN GJM1555C1H100GB01D -> 490-GJM1555C1H140FB01DCT-ND; MPN C5360816 -> GJM1555C1H140FB01D
- C56, C57, C59, C60: Digikey PN 1276-1043-1-ND -> 1276-1076-1-ND; MPN C1590 -> CL05A105KP5NNNC
- D12: MPN C84256 -> LTST-C281KGKT
- D5: MPN C2297 -> LTST-C281KGKT
- R10, R8: Digikey PN 311-1.50KLRCT-ND -> 311-1.20KLRCT-ND; MPN C22369819 -> RC0402FR-071K2L
- R17: Digikey PN P19181CT-ND -> 408-1447-1-ND
- R18, R7: Digikey PN 311-1.2KJRCT-ND -> 311-1.20KLRCT-ND; MPN C22369820 -> RC0402FR-071K2L
- R2: Digikey PN P100KLCT-ND -> RMCF0402JT10K0CT-ND; MPN C177329 -> RMCF0402JT10K0
- R37: value 32 -> 32k
- R6: Digikey PN 311-330LRCT-ND -> 311-1.20KLRCT-ND; MPN C177341 -> RC0402FR-071K2L
- U1: value (none) -> W25N01KVZEIR
- U12: value STM32F446ZCHx -> STM32F446ZCH6
- U2: value (none) -> ADXL375
- U4: value (none) -> ICM45686
- U7: value (none) -> BMP581
- U8: value (none) -> MMC5983MA
Connections:
- net +3.3V: now also C33.2, C35.2, C36.2, C37.1
- net GND: now also C35.1, C36.1, C37.2, C38.2, R39.1
- net VSENS_IN: now also C38.1
- new net: C33.1, R39.2
Other:
- moved on the sheet: C28, C32, R18, R26
