File: FIRM v1.0/FIRM_v1.0.kicad_sch (KiCad schematic)
At the start: 80 parts, among them J1 DM3CS-SF, J2 Conn_01x02_Pin, Q1 IRLML6402, U1 W25Q128JVS, U2 STM32F405RGTx, U3 ADXL371, U5 INA219AxDCN, U6 MIC5219-3.3YM5, U9 A-USBC-20F0-EA-GSR05, X1 32.768khz, Y1 12 MHz

Commit message: Reorg and Rename v1.0
Parts:
- U4, U7, U8: value ~ -> (none)
Connections:
- new net: U3.10 (RES), U3.13 (GND), U3.16 (GND)
