File: FIRM v2.0/FIRM_v2.0.kicad_sch (KiCad schematic)
At the start: 88 parts, among them J1 DM3CS-SF, J2 Conn_01x02_Pin, Q1 IRLML6402, U1 W25Q128JVS, U10 SAM-M10Q, U2 STM32F405RGTx, U3 ADXL371, U5 INA219AxDCN, U6 MIC5219-3.3YM5, U9 A-USBC-20F0-EA-GSR05, X1 32.768khz, Y1 12 MHz

Commit message: merge shoe to 2.0
Parts:
- added AE2: Antenna, symbol Device:Antenna
- added C35, C36, C37: 100n, Capacitor_SMD:C_0402_1005Metric, symbol Device:C
- added C38: 4u7, Capacitor_SMD:C_0402_1005Metric, symbol Device:C
- added C39: 0.1 uF, Capacitor_SMD:C_0402_1005Metric, symbol Device:C
- added C40: 10uF, Capacitor_SMD:C_0402_1005Metric, symbol Device:C
- added C41: 10nF, Capacitor_SMD:C_0402_1005Metric, symbol Device:C
- added D6: LED, symbol Device:LED
- added D7: CUHS20S60, diodes:CUHS20S60, symbol Device:D_Schottky
- added D8: LED, Diode_SMD:D_0402_1005Metric, symbol Device:LED
- added H4, H5, H6: MountingHole_Pad, MountingHole:MountingHole_2.2mm_M2_DIN965_Pad, symbol Mechanical:MountingHole_Pad
- added J3: Conn_01x22_Pin, symbol Connector:Conn_01x22_Pin
- added J4: Screw_Terminal_01x04, TerminalBlock:TerminalBlock_MaiXu_MX126-5.0-04P_1x04_P5.00mm, symbol Connector:Screw_Terminal_01x04
- added L2: 330 nH, symbol Device:L
- added M1, M3: (no value), transistors:TSM200N03D, symbol transistors:TSM200N03D
- added R19: 10k, symbol Device:R
- added R22, R29: 27k, Resistor_SMD:R_0402_1005Metric, symbol Device:R
- added R23, R24, R27, R28: 10k, Resistor_SMD:R_0402_1005Metric, symbol Device:R
- added R25, R30: 1.2k, Resistor_SMD:R_0402_1005Metric, symbol Device:R
- added R26, R31: 100k, Resistor_SMD:R_0402_1005Metric, symbol Device:R
- added R32: 100k, symbol Device:R
- added TSK_PS1240P02BT1: Buzzer, Buzzer_Beeper:Buzzer_TDK_PS1240P02BT_D12.2mm_H6.5mm, symbol Device:Buzzer
- added U12: SAM-M10Q, RF_GPS:ublox_SAM-M8Q, symbol RF_GPS:SAM-M8Q
- added U13: ~, sensors:E22-900MM22S, symbol sensors:E22-900MM22S
Connections:
- net +3.3V: now also C35.1, C36.1, C37.1, C38.1, C40.1, C41.1, J3.1 (Pin_1), R19.1, R32.1, U12.17 (VCC), U12.2 (VCC_IO), U12.3 (V_BCKP), U13.1 (VCC)
- net GND: now also C35.2, C36.2, C37.2, C38.2, C39.2, C40.2, C41.2, D6.1 (K), D8.1 (K), H4.1, H5.1, H6.1, J3.2 (Pin_2), L2.2, M3.1 (S1), M3.3 (S2), R22.2, R23.2, R24.2, R27.2, R28.2, R29.2, TSK_PS1240P02BT1.2 (-), U12.1 (GND), U12.10 (GND), U12.11 (GND), U12.15 (GND), U12.16 (GND), U12.20 (GND), U12.4 (GND), U12.5 (GND), U12.6 (GND), U13.16 (GND), U13.2 (GND), U13.7 (GND)
- net VBAT: now also D7.2 (A), J3.8 (Pin_8)
- new net: R19.2, U12.18 (~{RESET})
- new net: M1.1 (S1), M3.7 (D1), M3.8 (D1)
- new net: M1.3 (S2), M3.5 (D2), M3.6 (D2)
- new net: D8.2 (A), R30.2
- new net: C39.1, R32.2, U13.3 (NRST)
- new net: AE2.1 (A), L2.1, U13.6 (ANT)
- new net: D6.2 (A), R25.2
- new net: U3.10 (RES), U3.13 (GND), U3.16 (GND)
- new net +BATT: D7.1 (K), J4.2 (Pin_2), J4.4 (Pin_4)
- new net ARM_1: J3.11 (Pin_11), M3.2 (G1), R24.1
- new net ARM_2: J3.12 (Pin_12), M3.4 (G2), R28.1
- new net BUSY: J3.15 (Pin_15), U13.11 (BUSY)
- new net BUZZ: J3.22 (Pin_22), TSK_PS1240P02BT1.1 (+)
- new net FET_A: J4.1 (Pin_1), M1.7 (D1), M1.8 (D1), R25.1, R26.1
- new net FET_B: J4.3 (Pin_3), M1.5 (D2), M1.6 (D2), R30.1, R31.1
- new net FIRE_A: J3.9 (Pin_9), M1.2 (G1), R23.1
- new net FIRE_B: J3.10 (Pin_10), M1.4 (G2), R27.1
- new net MISO: J3.16 (Pin_16), U13.12 (MISO)
- new net MOSI: J3.17 (Pin_17), U13.13 (MOSI)
- new net NSS: J3.18 (Pin_18), U13.14 (NSS)
- new net RXEN: J3.20 (Pin_20), U13.9 (TXEN)
- new net SCK: J3.19 (Pin_19), U13.15 (SCK)
- new net SENS_A: J3.13 (Pin_13), R22.1, R26.2
- new net SENS_B: J3.14 (Pin_14), R29.1, R31.2
- new net SPI_MISO: J3.5 (Pin_5)
- new net SPI_MOSI: J3.6 (Pin_6)
- new net SPI_SCK: J3.7 (Pin_7)
- new net TXEN: J3.21 (Pin_21), U13.10 (RXEN)
- new net UART_RX: J3.3 (Pin_3), U12.13 (TXD)
- new net UART_TX: J3.4 (Pin_4), U12.14 (RXD)
- no-connect marks 26 -> 39
