File: FIRM v2.0/FIRM_v2.0.kicad_sch (KiCad schematic)
At the start: 88 parts, among them J1 DM3CS-SF, J2 Conn_01x02_Pin, Q1 IRLML6402, U1 W25Q128JVS, U10 SAM-M10Q, U2 STM32F405RGTx, U3 ADXL371, U5 INA219AxDCN, U6 MIC5219-3.3YM5, U9 A-USBC-20F0-EA-GSR05, X1 32.768khz, Y1 12 MHz

Commit message: Rename v2.0 Project
Parts:
- U11, U4, U7, U8: value ~ -> (none)
Connections:
- new net: U3.10 (RES), U3.13 (GND), U3.16 (GND)

Commit message: Updated Pinout for STM and migrated schematics from shoe to 2.0
Parts:
- removed C1, C13, C15, C17, C3, C6: 100n, Capacitor_SMD:C_0402_1005Metric, symbol Device:C
- removed C10, C5: 14p, Capacitor_SMD:C_0402_1005Metric, symbol Device:C
- removed C11, C12: 100n, Capacitor_SMD:C_0402_1005Metric, symbol Device:C_Small
- removed C14: 2u2, Capacitor_SMD:C_0402_1005Metric, symbol Device:C
- removed C16: 10n, Capacitor_SMD:C_0402_1005Metric, symbol Device:C
- removed C18: 1u, Capacitor_SMD:C_0402_1005Metric, symbol Device:C
- removed C2: 4u7, Capacitor_SMD:C_0402_1005Metric, symbol Device:C
- removed D1: LED_Blue, LED_SMD:LED_0402_1005Metric, symbol Device:LED
- removed D2: LED_Yellow, LED_SMD:LED_0402_1005Metric, symbol Device:LED
- removed D3: LED_Red, LED_SMD:LED_0402_1005Metric, symbol Device:LED
- removed FB1: 120 Ohms @ 100 MHz, Inductor_SMD:L_0603_1608Metric, symbol Device:FerriteBead
- removed J1: DM3CS-SF, connectors:HRS_DM3CS-SF, symbol connectors:DM3CS-SF
- removed R2: 47k, Resistor_SMD:R_0402_1005Metric, symbol Device:R_Small
- removed R3: 100k, Resistor_SMD:R_0402_1005Metric, symbol Device:R
- removed R8, R9: 330, symbol Device:R
- removed RN2: 10k, connectors:R_Array_YC104, symbol Device:R_Pack04
- removed TP12: SWDIO Through-Hole, connectors:Testpoint_1.5x1.5mm_1.0mm, symbol Connector:TestPoint
- removed TP13: SWCLK Through-Hole, connectors:Testpoint_1.5x1.5mm_1.0mm, symbol Connector:TestPoint
- removed TP14: 3.3V Test Point, connectors:Testpoint_1.5x1.5mm_1.0mm, symbol Connector:TestPoint
- removed TP5: PA10 Test Point, connectors:Testpoint_1.5x1.5mm_1.0mm, symbol Connector:TestPoint
- removed U1: W25Q128JVS, Package_SO:SOIC-8_5.3x5.3mm_P1.27mm, symbol Memory_Flash:W25Q128JVS
- removed U10: SAM-M10Q, RF_GPS:ublox_SAM-M8Q, symbol RF_GPS:SAM-M8Q
- removed U11: (no value), sensors:Wio_SX1262, symbol sensors:Wio_SX1262
- removed U2: STM32F405RGTx, Package_QFP:LQFP-64_10x10mm_P0.5mm, symbol MCU_ST_STM32F4:STM32F405RGTx
- removed X1: 32.768khz, connectors:Crystal_ECS-.327-6-12RR-TR, symbol Device:Crystal
- removed Y1: 12 MHz, connectors:Crystal_ECS-120-10-36B2-CWY-TR, symbol Device:Crystal_GND24
- added AE2: Antenna, symbol Device:Antenna
- added C1: 100n, Package_SO:SOIC-8_3.9x4.9mm_P1.27mm, symbol Device:C_Small
- added C12, C35, C36, C37, C39, C40, C41, C42, C43, C45, C48, C52, C54, C55: 100n, Capacitor_SMD:C_0402_1005Metric, symbol Device:C
- added C38: 4u7, Capacitor_SMD:C_0402_1005Metric, symbol Device:C
- added C44, C49, C51, C56, C57, C58, C59, C60: pad, Capacitor_SMD:C_0402_1005Metric, symbol Device:C_Small
- added C46, C47: 10p, Capacitor_SMD:C_0402_1005Metric, symbol Device:C
- added C50, C53: 2u2, Capacitor_SMD:C_0402_1005Metric, symbol Device:C
- added D10: LED_Yellow, LED_SMD:LED_0402_1005Metric, symbol Device:LED
- added D11: LED_Red, LED_SMD:LED_0402_1005Metric, symbol Device:LED
- added D6: LED, symbol Device:LED
- added D7: CUHS20S60, diodes:CUHS20S60, symbol Device:D_Schottky
- added D8: LED, Diode_SMD:D_0402_1005Metric, symbol Device:LED
- added D9: LED_Blue, LED_SMD:LED_0402_1005Metric, symbol Device:LED
- added J3: Screw_Terminal_01x04, TerminalBlock:TerminalBlock_MaiXu_MX126-5.0-04P_1x04_P5.00mm, symbol Connector:Screw_Terminal_01x04
- added L2: 330 nH, symbol Device:L
- added M1, M3: (no value), transistors:TSM200N03D, symbol transistors:TSM200N03D
- added R19: 10k, symbol Device:R
- added R2, R22, R23, R26, R27: 10k, Resistor_SMD:R_0402_1005Metric, symbol Device:R
- added R24, R29: 1.2k, Resistor_SMD:R_0402_1005Metric, symbol Device:R
- added R25, R30: 100k, Resistor_SMD:R_0402_1005Metric, symbol Device:R
- added R28: 27k, Resistor_SMD:R_0402_1005Metric, symbol Device:R
- added R3, R32, R33, R34, R9: 0, Package_DIP:DIP-8_W7.62mm, symbol Device:R_Small
- added R31: 100k, symbol Device:R
- added R8: 1k2, Resistor_SMD:R_0402_1005Metric, symbol Device:R_Small
- added RN1: 10k, Resistor_THT:R_Array_SIP6, symbol Device:R_Pack03
- added TP6: SWDIO Through-Hole, connectors:Testpoint_1.5x1.5mm_1.0mm, symbol Connector:TestPoint
- added TP7: SWCLK Through-Hole, connectors:Testpoint_1.5x1.5mm_1.0mm, symbol Connector:TestPoint
- added TSK_PS1240P02BT1: Buzzer, Buzzer_Beeper:Buzzer_TDK_PS1240P02BT_D12.2mm_H6.5mm, symbol Device:Buzzer
- added U1: (no value), Custom:W25N01GVZEIG, symbol Custom:W25N01GVZEIG
- added U10: ~, sensors:E22-900MM22S, symbol sensors:E22-900MM22S
- added U11: SAM-M10Q, RF_GPS:ublox_SAM-M8Q, symbol RF_GPS:SAM-M8Q
- added U12: STM32F446ZCHx, Package_BGA:UFBGA-144_7x7mm_Layout12x12_P0.5mm, symbol MCU_ST_STM32F4:STM32F446ZCHx
- added Y2: 12 MHz, Crystal:Crystal_SMD_3225-4Pin_3.2x2.5mm, symbol Device:Crystal_GND24
- C31: value 100n -> 0.1 uF; Digikey PN 1276-1043-1-ND -> 1276-1482-1-ND; MPN C1590 -> C1705
- C32: value 100n -> 10uF; Digikey PN 1276-1043-1-ND -> 1276-1482-1-ND; MPN C1590 -> C1705
- C33: value 100n -> 10nF; Digikey PN 1276-1043-1-ND -> 1276-1482-1-ND; MPN C1590 -> C1705
- C34: value 4u7 -> 100n; Digikey PN 1276-1482-1-ND -> 1276-1043-1-ND; MPN C1705 -> C1590
- C4: value 6p -> 4u7; Digikey PN 311-3714-1-ND -> 1276-1482-1-ND; MPN C37474 -> C1705
- C7: value 6p -> 100n; Digikey PN 311-3714-1-ND -> 1276-1043-1-ND; MPN C37474 -> C1590
- C9: value 2u2 -> 100n; Digikey PN 490-10012-1-ND -> 1276-1043-1-ND; MPN C1607 -> C1590
- R1: value 47k -> 0; footprint Resistor_SMD:R_0402_1005Metric -> Package_DIP:DIP-8_W7.62mm; Digikey PN 311-47.0KLRCT-ND -> (none); MPN C22356633 -> (none)
- R10: value 10k -> 27k; footprint (none) -> Resistor_SMD:R_0402_1005Metric
- R11, R12: value 3k3 -> 0; footprint Resistor_SMD:R_0402_1005Metric -> Package_DIP:DIP-8_W7.62mm; Digikey PN P3.3KDCCT-ND -> (none); MPN C22356633 -> (none)
- R13: value 330 -> 0; footprint Resistor_SMD:R_0402_1005Metric -> Package_DIP:DIP-8_W7.62mm; Digikey PN 311-330LRCT-ND -> (none); MPN C177341 -> (none)
- R14: value 1k2 -> 0; footprint Resistor_SMD:R_0402_1005Metric -> Package_DIP:DIP-8_W7.62mm; Digikey PN 311-1.2KJRCT-ND -> (none); MPN C22369820 -> (none)
- R15: value 1k5 -> 0; footprint Resistor_SMD:R_0402_1005Metric -> Package_DIP:DIP-8_W7.62mm; Digikey PN 311-1.50KLRCT-ND -> (none); MPN C22369819 -> (none)
- R4, R5: value 47k -> 3k3; footprint Resistor_SMD:R_0402_1005Metric -> Package_DIP:DIP-8_W7.62mm; Digikey PN 311-47.0KLRCT-ND -> (none); MPN C22356633 -> (none)
- R6: value 47k -> 1.2k; Digikey PN 311-47.0KLRCT-ND -> 311-330LRCT-ND; MPN C22356633 -> C177341
- R7: value 47k -> 1k2; Digikey PN 311-47.0KLRCT-ND -> 311-1.2KJRCT-ND; MPN C22356633 -> C22369820
- TP1: value PA0 Test Point -> 3.3V Test Point
- TP2: value PA1 Test Point -> GND Test Point
- TP3: value PA2 Test Point -> UART_RX Test Point
- TP4: value PA9 Test Point -> UART_TX Test Point
Connections:
- net LSE_IN is gone; now on net +3.3V: C4.1
- net LSE_OUT is gone; now on net +3.3V: C7.1
- net PA0 is gone; now on net +3.3V: TP1.1
- net PA1 is gone; now on net GND: TP2.1
- net SDIO_CMD is gone; now on net I2C1_SDA: R4.1
- net SDIO_D0 is gone; now on net I2C1_SCL: R5.1
- net VCAP1 is gone; now on net +3.3V: C9.1
- net +3.3V: now also C1.1, C12.1, C35.1, C36.1, C37.1, C38.1, C39.1, C40.1, C41.1, C42.1, C43.1, C48.1, C52.1, C54.1, C55.1, R19.1, R31.1, RN1.1 (R1.1), RN1.2 (R2.1), RN1.3 (R3.1), U1.8 (VCC), U10.1 (VCC), U11.17 (VCC), U11.2 (VCC_IO), U11.3 (V_BCKP), U12.C11 (VDDUSB), U12.C2 (VBAT), U12.D3 (VDD), U12.E5 (PDR_ON), U12.F10 (VDD), U12.F4 (VDD), U12.F5 (VDD), U12.F6 (VDD), U12.F7 (VDD), U12.F8 (VDD), U12.F9 (VDD), U12.G5 (VDD), U12.G6 (VDD), U12.G7 (VDD), U12.M1 (VDDA); no longer C31.1, R1.2, R10.1, R11.2, R12.2, R6.2, R7.2
- net BMP_CS: now also U12.L11 (PB14)
- net BMP_INT: now also U12.M2 (PA3)
- net GND: now also R10.2, C1.2, C12.2, C35.2, C36.2, C37.2, C38.2, C39.2, C40.2, C41.2, C42.2, C43.2, C44.1, C45.2, C46.2, C47.2, C48.2, C49.1, C50.2, C51.1, C52.2, C53.2, C54.2, C55.2, C56.1, C57.1, C58.1, C59.1, C60.1, D10.1 (K), D11.1 (K), D6.1 (K), D8.1 (K), D9.1 (K), L2.2, M3.1 (S1), M3.3 (S2), R2.2, R22.2, R23.2, R26.2, R27.2, R28.2, TSK_PS1240P02BT1.2 (-), U1.4 (GND), U1.9 (EP), U10.16 (GND), U10.2 (GND), U10.7 (GND), U11.1 (GND), U11.10 (GND), U11.11 (GND), U11.15 (GND), U11.16 (GND), U11.20 (GND), U11.4 (GND), U11.5 (GND), U11.6 (GND), U12.D2 (VSS), U12.E6 (VSS), U12.E7 (VSS), U12.G10 (VSS), U12.G4 (VSS), U12.G8 (VSS), U12.H5 (BYPASS_REG), U12.H6 (VSS), U12.J1 (VSSA), Y2.2, Y2.4
- net HIG_CS: now also U12.G11 (PG8)
- net HIG_INT: now also U12.K2 (PA1)
- net I2C1_SCL: now also U12.C5 (PB8); no longer R11.1
- net I2C1_SDA: now also U12.B5 (PB9); no longer R12.1
- net IMU_CS: now also U12.B2 (PE4)
- net IMU_INT: now also U12.L4 (PB0)
- net MAG_CS: now also U12.J11 (PG3)
- net MAG_INT: now also U12.L2 (PA2)
- net MISO2: now also C59.2, R3.1; no longer U3.7 (MISO)
- net MOSI2: now also R1.2, C56.2; no longer U3.6 (MOSI)
- net NRST: now also C45.1, U12.F1 (NRST)
- net SCK2: now also R33.2; no longer U3.4 (SCLK)
- net USB_D+: now also U12.B12 (PA12)
- net USB_D-: now also U12.C12 (PA11)
- net VBAT: now also D7.2 (A)
- net at R14.1: now also U12.E11 (PC9)
- net at R15.1: now also U12.C10 (PC12)
- net at R13.1: now also U12.G2 (PF9)
- net DBUG_0 renamed QUADSPI_BK1_IO1
- net QUADSPI_BK1_IO1: now also C44.2, U1.2 (DO(IO1))
- net DBUG_1 renamed QUADSPI_BK1_IO0
- net QUADSPI_BK1_IO0: now also C60.2, U1.5 (DI(IO0))
- net DBUG_2 renamed SCK3
- net SCK3: now also U3.4 (SCLK), U10.15 (SCK)
- net PA2 renamed USART1_RX
- net USART1_RX: now also U12.D6 (PB7)
- net PA9 renamed USART1_TX
- net USART1_TX: now also U12.C6 (PB6)
- net SDIO_D1: no longer names the net of R6.1
- net SDIO_D1: now also D9.2 (A)
- net SDIO_D2: no longer names the net of R1.1
- net SDIO_D2: now also U12.H2 (PC1)
- net SD_DETECT: no longer names the net of R7.1
- net SD_DETECT: now also D10.2 (A)
- new net: AE2.1 (A), L2.1, U10.6 (ANT)
- new net: M1.1 (S1), M3.7 (D1), M3.8 (D1)
- new net: M1.3 (S2), M3.5 (D2), M3.6 (D2)
- new net: R19.2, U11.18 (~{RESET})
- new net: R2.1, U12.D5 (BOOT0)
- new net: R34.1, U12.J9 (PD10)
- new net: D8.2 (A), R29.2
- new net: R9.1, U12.B10 (PC11)
- new net: R33.1, U12.D9 (PD3)
- new net: R12.1, U12.F2 (PF7)
- new net: R11.2, U12.F3 (PF6)
- new net: C53.1, U12.G9 (VCAP_2)
- new net: R3.2, U12.H3 (PC2)
- new net: C50.1, U12.H7 (VCAP_1)
- new net: R32.1, U12.J5 (PB2)
- new net: C31.1, R31.2, U10.3 (NRST)
- new net: U3.10 (RES), U3.13 (GND), U3.16 (GND)
- new net: D11.2 (A), R8.1
- new net: D6.2 (A), R24.2
- new net +BATT: D7.1 (K), J3.2 (Pin_2), J3.4 (Pin_4)
- new net ARM_1: M3.2 (G1), R23.1
- new net ARM_2: M3.4 (G2), R27.1
- new net BUSY: U10.11 (BUSY)
- new net BUZZ: TSK_PS1240P02BT1.1 (+)
- new net DEBUG0: U12.A3 (PE2)
- new net DEBUG1: U12.A4 (PE1)
- new net DEBUG2: U12.A2 (PE3)
- new net DEBUG_0: R6.2
- new net DEBUG_1: R7.2
- new net DEBUG_2: R8.2
- new net FET_A: J3.1 (Pin_1), M1.7 (D1), M1.8 (D1), R24.1, R25.1
- new net FET_B: J3.3 (Pin_3), M1.5 (D2), M1.6 (D2), R29.1, R30.1
- new net FIRE_A: M1.2 (G1), R22.1
- new net FIRE_B: M1.4 (G2), R26.1
- new net MISO3: C57.2, R9.2, U10.12 (MISO), U3.7 (MISO)
- new net MOSI3: C58.2, R34.2, U10.13 (MOSI), U3.6 (MOSI)
- new net NSS: U10.14 (NSS)
- new net QUADSPI_BK1_IO2: C49.2, R12.2, RN1.5 (R2.2), U1.3 (/WP(IO2))
- new net QUADSPI_BK1_IO3: C51.2, R11.1, RN1.6 (R1.2), U1.7 (/HOLD(IO3))
- new net QUADSPI_BK1_NCS: RN1.4 (R3.2), U1.1 (/CS), U12.H11 (PG6)
- new net QUADSPI_CLK: R32.2, U1.6 (CLK)
- new net RCC_OSC_IN: C46.1, U12.D1 (PH0), Y2.1
- new net RCC_OSC_OUT: C47.1, U12.E1 (PH1), Y2.3
- new net RXEN: U10.9 (TXEN)
- new net SENS_A: R10.1, R25.2
- new net SENS_B: R28.1, R30.2
- new net SYS_JTCK-SWCLK: TP7.1, U12.A11 (PA14)
- new net SYS_JTMS-SWDIO: TP6.1, U12.A12 (PA13)
- new net TXEN: U10.10 (RXEN)
- new net UART2_RX: U11.13 (TXD)
- new net UART2_TX: U11.14 (RXD)
- new net USART2_RX: U12.A8 (PD6)
- new net USART2_TX: U12.B9 (PD5)
- no-connect marks 26 -> 33
Other:
- company: Seth O, Will S, Harshil M, Jackson E -> Emmanuel RM, Will S, William D
- title: FIRM -> FIRM 2.0

Commit message: Wired up MIC216 and a third DEBUG LED
Parts:
- removed C19, C20: 100n, Capacitor_SMD:C_0402_1005Metric, symbol Device:C_Small
- removed C26: 470p, Capacitor_SMD:C_0402_1005Metric, symbol Device:C_Small
- removed R16: 100k, Resistor_SMD:R_0402_1005Metric, symbol Device:R
- removed R18: 1k2, Resistor_SMD:R_0402_1005Metric, symbol Device:R_Small
- removed R20, R21: 5.1k, Resistor_SMD:R_0402_1005Metric, symbol Device:R
- removed U3: ADXL371, Sensor_Motion:Analog_LGA-16_3.25x3mm_P0.5mm_LayoutBorder3x5y, symbol Sensor_Motion:ADXL363
- removed U6: MIC5219-3.3YM5, Package_TO_SOT_SMD:SOT-23-5, symbol Regulator_Linear:MIC5219-3.3YM5
- added C2, C3: 100n, HPRC_Sensors:ADXL375BCCZ-RL7, symbol Device:C_Small
- added D12: LED_Red, LED_SMD:LED_0402_1005Metric, symbol Device:LED
- added R16: 0, Package_DIP:DIP-8_W7.62mm, symbol Device:R_Small
- added R18: 10m, Resistor_SMD:R_0402_1005Metric, symbol Device:R
- added R20: 100k, Resistor_SMD:R_0402_1005Metric, symbol Device:R_Small
- added R21: 1k2, Resistor_SMD:R_0402_1005Metric, symbol Device:R_Small
- added R35, R36: 5.1k, Resistor_SMD:R_0402_1005Metric, symbol Device:R
- added U2: (no value), HPRC_Sensors:ADXL375BCCZ-RL7, symbol HPRC_Sensors:ADXL375
- added U3: (no value), HPRC_regulators:MIC5216-3.3M5, symbol HPRC_Regulators:MIC5216-3.3YM5-TR
- R11: value 0 -> 1k2; footprint Package_DIP:DIP-8_W7.62mm -> Resistor_SMD:R_0402_1005Metric; Digikey PN (none) -> 311-1.50KLRCT-ND; MPN (none) -> C22369819
- R17: value 10m -> 100k; Digikey PN P19181CT-ND -> P100KLCT-ND; MPN (none) -> C177329
Connections:
- net +3.3V: now also C2.1, C3.1, R21.2, U2.1 (VDD_I/0), U2.12 (SDO/ALT_ADD), U2.6 (Vs), U2.7 (CS), U3.5 (OUT)
- net DEBUG0: now also U12.A4 (PE1); no longer U12.A3 (PE2)
- net DEBUG1: now also U12.A3 (PE2); no longer U12.A4 (PE1)
- net GND: now also R17.2, C2.2, C3.2, D12.1 (K), R35.2, R36.2, U2.2 (GND), U2.4 (GND), U2.5 (GND), U3.2 (GND)
- net HIG_INT: now also U2.9 (INT1)
- net I2C1_SDA: now also U2.13 (SDA/SDI/SDIO)
- net QUADSPI_BK1_IO0: now also R16.2; no longer R14.2
- net QUADSPI_BK1_IO1: now also R14.2; no longer R13.2
- net QUADSPI_BK1_IO2: now also R13.2; no longer R12.2
- net QUADSPI_BK1_IO3: now also R12.1; no longer R11.1
- net VBUS: now also R17.1
- net VSENS_IN: now also R18.1; no longer R17.1
- net VSENS_OUT: now also R18.2, R20.2, U3.1 (IN), U3.3 (EN); no longer R17.2
- net at U9.A5 (CC1): now also R35.1
- net at U9.B5 (CC2): now also R36.1
- net at D5.2 (A): now also R21.1
- net DEBUG3: now reaches U12.A1 (PC13)
- net DEBUG3: now also R11.2
- net at R14.1: now also U12.G2 (PF9); no longer U12.E11 (PC9)
- net at U12.F2 (PF7): now also R13.1; no longer R12.1
- net at U12.F3 (PF6): now also R12.2; no longer R11.2
- new net: R16.1, U12.E11 (PC9)
- new net: D12.2 (A), R11.1
- new net I2C1_SDL: U2.14 (SCL/SCLK)
- new net MIC_FLAG: R20.1, U3.4 (FLG)
- no-connect marks 33 -> 30

Commit message: Update FIRM 2.0 with new changes to flash, ADXL, and Voltage reg
Parts:
- removed R35, R36: 5.1k, Resistor_SMD:R_0402_1005Metric, symbol Device:R
- removed RN1: 10k, Resistor_THT:R_Array_SIP6, symbol Device:R_Pack03
- removed U1: (no value), Custom:W25N01GVZEIG, symbol Custom:W25N01GVZEIG
- added R35, R36, R37: 10k, Resistor_SMD:R_0402_1005Metric, symbol Device:R_Small
- added R38, R39: 5.1k, Resistor_SMD:R_0402_1005Metric, symbol Device:R
- added U1: (no value), HPRC_Storage:W25N01KVZEIR, symbol HPRC_Storage:W25N01KVZEIR
- C1: footprint Package_SO:SOIC-8_3.9x4.9mm_P1.27mm -> Capacitor_SMD:C_0402_1005Metric
- C2, C3: footprint HPRC_Sensors:ADXL375BCCZ-RL7 -> Capacitor_SMD:C_0402_1005Metric
- C44, C49, C51, C56, C57, C58, C59, C60: now not fitted
- R12, R13, R14, R16, R3, R32, R4, R5: footprint Package_DIP:DIP-8_W7.62mm -> Resistor_SMD:R_0402_1005Metric
- R19, R31: footprint (none) -> Resistor_SMD:R_0402_1005Metric
Connections:
- net +3.3V: now also R35.2, R36.2, R37.2, U1.8 (VCC)
- net GND: now also R38.2, R39.2, U1.4 (GND), U1.9 (EP)
- net QUADSPI_BK1_IO0: now also U1.5 (DI(IO0))
- net QUADSPI_BK1_IO1: now also U1.2 (DO(IO1))
- net QUADSPI_BK1_IO2: now also R36.1, U1.3 (/WP(IO2))
- net QUADSPI_BK1_IO3: now also R35.1, U1.7 (/HOLD(IO3))
- net QUADSPI_BK1_NCS: now also R37.1, U1.1 (/CS)
- net QUADSPI_CLK: now also U1.6 (CLK)
- net at U9.A5 (CC1): now also R38.1
- net at U9.B5 (CC2): now also R39.1
- net DEBUG3 renamed DEBUG_3

Commit message: Added SCH16T-K01-1 IMU to FIRM2.0
Parts:
- added C61, C65: 100n, Capacitor_SMD:C_0402_1005Metric, symbol Device:C_Small
- added C62: 10u, Capacitor_SMD:C_0402_1005Metric, symbol Device:C_Small
- added C63, C64: 1u, Capacitor_SMD:C_0402_1005Metric, symbol Device:C_Small
- added R40: 10k, Resistor_SMD:R_0402_1005Metric, symbol Device:R
- added U13: SCH16T-K01-10, HPRC_Sensors:XDCR_SCH16T-K01-10, symbol HPRC_Sensors:SCH16T-K01-10
Connections:
- net +3.3V: now also C61.1, C64.1, C65.1, R40.1, U13.17 (V3P3), U13.18 (VDDIO), U13.8 (V3P3)
- net GND: now also C61.2, C62.2, C63.2, C64.2, C65.2, U13.1 (HEATSINK), U13.12 (GND), U13.13 (GND), U13.16 (GND), U13.24 (HEATSINK), U13.3 (TA9), U13.4 (TA8), U13.5 (RESERVED), U13.7 (RESERVED), U13.9 (GND)
- net MISO3: now also U13.19 (MISO)
- net MOSI3: now also U13.23 (MOSI)
- net SCK3: now also U13.21 (SCK)
- net IMUL_INT: now reaches U12.K10 (PD13)
- net IMUL_INT: now also U13.20 (DRY_SYNC)
- net IMUL_CS: now reaches U12.K11 (PD14)
- net IMUL_CS: now also U13.22 (CS)
- new net: C62.1, U13.10 (VREGA2), U13.11 (VREGA)
- new net: C63.1, U13.14 (VREGD2), U13.15 (VREGD)
- new net: R40.2, U13.6 (~{EXTRES})
- no-connect marks 30 -> 31

Commit message: Moved new Pyros to FIRM 2.0
Parts:
- removed C2: 100n, Capacitor_SMD:C_0402_1005Metric, symbol Device:C_Small
- removed C24: 10u, Capacitor_SMD:C_0402_1005Metric, symbol Device:C_Small
- removed C56, C57, C58, C59, C60: pad, Capacitor_SMD:C_0402_1005Metric, symbol Device:C_Small
- removed D4: D_Schottky, connectors:D_schottky_NSR05F30NXT5G, symbol Device:D_Schottky
- removed D6: LED, symbol Device:LED
- removed D7: CUHS20S60, diodes:CUHS20S60, symbol Device:D_Schottky
- removed D8: LED, Diode_SMD:D_0402_1005Metric, symbol Device:LED
- removed J3: Screw_Terminal_01x04, TerminalBlock:TerminalBlock_MaiXu_MX126-5.0-04P_1x04_P5.00mm, symbol Connector:Screw_Terminal_01x04
- removed M1, M3: (no value), transistors:TSM200N03D, symbol transistors:TSM200N03D
- removed Q1: IRLML6402, Package_TO_SOT_SMD:SOT-23, symbol Transistor_FET:IRLML6402
- removed R10, R28: 27k, Resistor_SMD:R_0402_1005Metric, symbol Device:R
- removed R16: 0, Resistor_SMD:R_0402_1005Metric, symbol Device:R_Small
- removed R18: 10m, Resistor_SMD:R_0402_1005Metric, symbol Device:R
- removed R20: 100k, Resistor_SMD:R_0402_1005Metric, symbol Device:R_Small
- removed R21: 1k2, Resistor_SMD:R_0402_1005Metric, symbol Device:R_Small
- removed R22, R23, R26, R27, R40: 10k, Resistor_SMD:R_0402_1005Metric, symbol Device:R
- removed R24, R29: 1.2k, Resistor_SMD:R_0402_1005Metric, symbol Device:R
- removed R30: 100k, Resistor_SMD:R_0402_1005Metric, symbol Device:R
- removed R38, R39: 5.1k, Resistor_SMD:R_0402_1005Metric, symbol Device:R
- removed TP1: 3.3V Test Point, connectors:Testpoint_1.5x1.5mm_1.0mm, symbol Connector:TestPoint
- removed TP2: GND Test Point, connectors:Testpoint_1.5x1.5mm_1.0mm, symbol Connector:TestPoint
- removed TP3: UART_RX Test Point, connectors:Testpoint_1.5x1.5mm_1.0mm, symbol Connector:TestPoint
- removed TP4: UART_TX Test Point, connectors:Testpoint_1.5x1.5mm_1.0mm, symbol Connector:TestPoint
- removed TP6: SWDIO Through-Hole, connectors:Testpoint_1.5x1.5mm_1.0mm, symbol Connector:TestPoint
- removed TP7: SWCLK Through-Hole, connectors:Testpoint_1.5x1.5mm_1.0mm, symbol Connector:TestPoint
- removed U3: (no value), HPRC_regulators:MIC5216-3.3M5, symbol HPRC_Regulators:MIC5216-3.3YM5-TR
- removed U4: (no value), sensors:IC_ICM-45686, symbol sensors:ICM-45686
- removed U7: (no value), sensors:BMPFootprintNoSolderMask, symbol sensors:BMP581
- removed U8: (no value), sensors:IC_MMC5983MA, symbol sensors:MMC5983MA
- removed U9: A-USBC-20F0-EA-GSR05, connectors:A-USBC-20F0-EA-GSR05, symbol connectors:A-USBC-20F0-EA-GSR05
- removed Y2: 12 MHz, Crystal:Crystal_SMD_3225-4Pin_3.2x2.5mm, symbol Device:Crystal_GND24
- added C26: 10u, Capacitor_SMD:C_1206_3216Metric, symbol Device:C_Small
- added C56, C57, C59, C60: 1u, Capacitor_SMD:C_0402_1005Metric, symbol Device:C
- added C58: 100n, Capacitor_SMD:C_0402_1005Metric, symbol Device:C
- added C66: 100n, Capacitor_SMD:C_0402_1005Metric, symbol Device:C_Small
- added D13: LED, symbol Device:LED
- added D14: CUHS20S60, diodes:CUHS20S60, symbol Device:D_Schottky
- added D15: LED, Diode_SMD:D_0402_1005Metric, symbol Device:LED
- added J1: Pin, Connector_PinHeader_1.00mm:PinHeader_1x06_P1.00mm_Vertical, symbol Connector:Conn_01x06_Pin
- added J4: Screw_Terminal_01x04, TerminalBlock:TerminalBlock_MaiXu_MX126-5.0-04P_1x04_P5.00mm, symbol Connector:Screw_Terminal_01x04
- added L1: 2u2, Inductor_SMD:L_1008_2520Metric, symbol Device:L_Small
- added PS1: TPS62162DSGR, HPRC_Regulators:TPS62162DSGR, symbol HPRC_Regulators:TPS62162DSGR
- added Q1: DMP3098L-7, HPRC_Logic:DMP3098L-7, symbol HPRC_Logic_ICs:DMP3098L-7
- added Q2, Q3: G120N02D32, HPRC_Transistors:G120N02D32, symbol HPRC_Transistors:G120N02D32
- added R10, R18: 1k2, Resistor_SMD:R_0402_1005Metric, symbol Device:R_Small
- added R20, R21: 5.1k, Resistor_SMD:R_0402_1005Metric, symbol Device:R
- added R22, R23, R24, R55: 10k, Resistor_SMD:R_0402_1005Metric, symbol Device:R_Small
- added R26, R27, R29, R38: 100k, Resistor_SMD:R_0402_1005Metric, symbol Device:R_Small
- added R28: 80k, Resistor_SMD:R_0402_1005Metric, symbol Device:R_Small
- added R30: 7k6, Resistor_SMD:R_0402_1005Metric, symbol Device:R_Small
- added R39: 0, Resistor_SMD:R_0201_0603Metric, symbol Device:R_Small
- added R40: 1k, Resistor_SMD:R_0402_1005Metric, symbol Device:R_Small
- added R41, R52: 27k, Resistor_SMD:R_0402_1005Metric, symbol Device:R
- added R42, R43, R48, R49: 10k, Resistor_SMD:R_0402_1005Metric, symbol Device:R
- added R44, R45, R50, R51: 220, Resistor_SMD:R_0402_1005Metric, symbol Device:R
- added R46, R53: 1.2k, Resistor_SMD:R_0402_1005Metric, symbol Device:R
- added R47, R54: 100k, Resistor_SMD:R_0402_1005Metric, symbol Device:R
- added U3: TPS2121RUXR, HPRC_Regulators:IC_TPS2121RUXR, symbol HPRC_Regulators:TPS2121RUXR
- added U4: ICM45686, HPRC_Sensors:IC_ICM-45686, symbol HPRC_Sensors:ICM-45686
- added U7: BMP581, HPRC_Sensors:BMP581, symbol HPRC_Sensors:BMP581
- added U8: MMC5983MA, HPRC_Sensors:IC_MMC5983MA, symbol HPRC_Sensors:MMC5983MA
- added U9: A-USBC-20F0-EA-GSR05, HPRC_Connectors:A-USBC-20F0-EA-GSR05, symbol HPRC_Connectors:A-USBC-20F0-EA-GSR05
- added Y1: 12 MHz, HPRC_Connectors:Crystal_ECS-120-10-36B2-CWY-TR, symbol Device:Crystal_GND24
- C28: footprint Capacitor_SMD:C_0402_1005Metric -> Capacitor_SMD:C_0603_1608Metric; Digikey PN 1276-1451-1-ND -> 490-12737-1-ND; MPN C1691 -> GRM188R61E106MA73J
- C44: value pad -> 10u; footprint Capacitor_SMD:C_0402_1005Metric -> Capacitor_SMD:C_0603_1608Metric; Digikey PN 1276-1043-1-ND -> 490-12737-1-ND; MPN C1590 -> GRM188R61E106MA73J; now fitted
- C46, C47: value 10p -> 14p; MPN C5360816 -> GJM1555C1H140FB01D
- C49: value pad -> 1u; Digikey PN 1276-1043-1-ND -> 1276-1067-1-ND; MPN C1590 -> C1592; now fitted
- C51: value pad -> 22u; footprint Capacitor_SMD:C_0402_1005Metric -> Capacitor_SMD:C_1210_3225Metric; Digikey PN 1276-1043-1-ND -> 490-GRM32ER71E226KE15KCT-ND; MPN C1590 -> GRM32ER71E226KE15K; now fitted
- C61: value 100n -> 22u; footprint Capacitor_SMD:C_0402_1005Metric -> Capacitor_SMD:C_0603_1608Metric; Digikey PN (none) -> 1276-2867-1-ND; MPN (none) -> CL10A226KQ8NRNE
- C62: value 10u -> 100n; Digikey PN (none) -> 1276-1043-1-ND; MPN (none) -> C1590
- C63: value 1u -> 10u
- C65: value 100n -> 1u; Digikey PN (none) -> 1276-1067-1-ND; MPN (none) -> C1592
- D12: value LED_Red -> LED_Green; Digikey PN 160-LTST-C281KRKTCT-ND -> 160-LTST-C281KGKTCT-ND; MPN C84256 -> LTST-C281KGKT
- D5: MPN C2297 -> LTST-C281KGKT
- J2: value Conn_01x02_Pin -> Vbat Jmpr; footprint connectors:power_headers -> HPRC_Connectors:power_headers
- R1, R15, R33, R34, R9: footprint Package_DIP:DIP-8_W7.62mm -> Resistor_SMD:R_0201_0603Metric
- R11: value 1k2 -> 0; footprint Resistor_SMD:R_0402_1005Metric -> Resistor_SMD:R_0201_0603Metric; Digikey PN 311-1.50KLRCT-ND -> (none); MPN C22369819 -> (none)
- R12, R13, R14, R3, R32: footprint Resistor_SMD:R_0402_1005Metric -> Resistor_SMD:R_0201_0603Metric
- R17: value 100k -> 100m; Digikey PN P100KLCT-ND -> 408-1447-1-ND; MPN C177329 -> (none)
- R2: Digikey PN P100KLCT-ND -> RMCF0402JT10K0CT-ND; MPN C177329 -> RMCF0402JT10K0
- R25: value 100k -> 10k
- R35: value 10k -> 57.6k
- R36: value 10k -> 5.1k
- R37: value 10k -> 32k
- R6: Digikey PN 311-330LRCT-ND -> 311-1.20KLRCT-ND; MPN C177341 -> RC0402FR-071K2L
- R7: Digikey PN 311-1.2KJRCT-ND -> 311-1.20KLRCT-ND; MPN C22369820 -> RC0402FR-071K2L
- R8: Digikey PN 311-1.50KLRCT-ND -> 311-1.20KLRCT-ND; MPN C22369819 -> RC0402FR-071K2L
- U1: value (none) -> W25N01KVZEIR
- U12: value STM32F446ZCHx -> STM32F446ZCH6
- U2: value (none) -> ADXL375
Connections:
- net DEBUG0 is gone; now on net DEBUG_0: U12.A4 (PE1)
- net DEBUG1 is gone; now on net DEBUG_1: U12.A3 (PE2)
- net DEBUG2 is gone; now on net DEBUG_2: U12.A2 (PE3)
- net I2C1_SDL is gone; now on net I2C1_SCL: U2.14 (SCL/SCLK)
- net +3.3V: now also C49.2, C62.2, R25.1, R37.1, U12.L1 (VREF+), C56.1, C57.1, C58.1, C59.1, C66.2, J1.6 (Pin_6), L1.2, PS1.6 (VOS), R18.2, R22.2, R23.2, R24.2, R26.1, U4.5 (VDDIO), U4.8 (VDD), U7.1 (VDDIO), U7.10 (VDD), U8.13 (VDDIO), U8.2 (VDD); no longer C28.1, C64.1, R35.2, R36.2, R37.2
- net +BATT: now also D14.1 (K), J4.2 (Pin_2), J4.4 (Pin_4)
- net ARM_1: now also R43.1, R45.2
- net ARM_2: now also R49.1, R51.2
- net BMP_CS: now also U7.6 (CSB)
- net BMP_INT: now also U7.7 (INT)
- net DEBUG_3: now also R10.2; no longer R11.2
- net FET_A: now also J4.1 (Pin_1), Q2.7 (D1), Q2.8 (D1), R46.1, R47.1; no longer R25.1
- net FET_B: now also J4.3 (Pin_3), Q2.5 (D2), Q2.6 (D2), R53.1, R54.1
- net FIRE_A: now also R42.1, R44.2
- net FIRE_B: now also R48.1, R50.2
- net GND: now also C44.2, C51.2, C62.1, R35.2, U12.K1 (VREF-), C26.2, C56.2, C57.2, C58.2, C59.2, C60.2, C66.1, D13.1 (K), D14.2 (A), D15.1 (K), J1.5 (Pin_5), PS1.1 (PGND), PS1.4 (AGND), PS1.5 (FB), PS1.9 (EXP), Q1.2, Q3.1 (S1), Q3.3 (S2), R20.2, R21.2, R27.2, R29.1, R30.2, R38.2, R39.1, R40.2, R41.2, R42.2, R43.2, R48.2, R49.2, R52.2, R55.2, U3.12 (GND), U3.2 (IN2), U3.2_1 (IN2), U3.5 (OV1), U3.9 (ST), U4.6 (GND), U7.3 (VSS), U7.8 (VSS), U7.9 (VSS), U8.11 (GND), U8.9 (GND), U9.A1 (GND), U9.B1 (GND), U9.S1 (SHIELD), Y1.2 (G), Y1.4 (G); no longer C49.1, C51.1, C62.2, R17.2
- net HIG_INT: now also U2.8 (INT1); no longer U2.9 (INT1)
- net IMU_CS: now also U4.12 (AP_CS)
- net IMU_INT: now also U4.4 (INT1/INT)
- net MAG_CS: now also U8.4 (SPI_CS)
- net MAG_INT: now also U8.15 (INT)
- net MISO2: now also U4.1 (AP_SDO/AP_AD0), U7.5 (SDO), U8.5 (SPI_SDO)
- net MOSI2: now also U4.14 (AP_SDA/APSDIO/APSDI), U7.4 (SDI), U8.16 (SDA/ SPI_SDI)
- net QUADSPI_BK1_IO0: now also R14.2
- net QUADSPI_BK1_IO1: now also R13.2; no longer C44.2, R14.2
- net QUADSPI_BK1_IO2: now also R12.2, R23.1; no longer C49.2, R13.2, R36.1
- net QUADSPI_BK1_IO3: now also R11.1, R24.1; no longer C51.2, R12.1, R35.1
- net QUADSPI_BK1_NCS: now also R22.1; no longer R37.1
- net RCC_OSC_IN: now also Y1.1
- net RCC_OSC_OUT: now also Y1.3
- net SCK2: now also U4.13 (AP_SCL/AP_SCLK), U7.2 (SCK), U8.1 (SCL/ SPI_SCK)
- net SENS_A: now also R41.1, R47.2; no longer R25.2
- net SENS_B: now also R52.1, R54.2
- net SYS_JTCK-SWCLK: now also J1.3 (Pin_3)
- net SYS_JTMS-SWDIO: now also J1.4 (Pin_4)
- net USART1_RX: now also J1.2 (Pin_2)
- net USART1_TX: now also J1.1 (Pin_1)
- net USB_D+: now also U9.A6 (D+), U9.B6 (D+)
- net USB_D-: now also U9.A7 (D-), U9.B7 (D-)
- net VBUS: now also C28.1, R36.1, R28.1, U3.7 (IN1), U3.7_1 (IN1), U9.A4 (VBUS), U9.B4 (VBUS); no longer R17.1
- net VSENS_IN: now also C51.1, R17.1, U3.1 (OUT), U3.1_1 (OUT), U3.8 (OUT), U3.8_1 (OUT)
- net VSENS_OUT: now also R17.2, C26.1, PS1.2 (VIN), PS1.3 (EN)
- net at U13.10 (VREGA2), U13.11 (VREGA): now also C63.1; no longer C62.1
- net at D12.2 (A): now also R10.1; no longer R11.1
- net at C30.2: now also U8.10 (CAP)
- net at U12.B11 (PC10): now also R15.1
- net at U12.C10 (PC12): now also R34.1; no longer R15.1
- net USB_SENS: now reaches U12.D12 (PA9)
- net USB_SENS: now also R36.2, R55.1
- net at U12.E11 (PC9): now also R14.1
- net at U12.F2 (PF7): now also R12.1; no longer R13.1
- net at U12.F3 (PF6): now also R11.2; no longer R12.2
- net at U12.G2 (PF9): now also R13.1; no longer R14.1
- net at U12.J9 (PD10): no longer R34.1
- net at D5.2 (A): now also R18.1
- net at U13.14 (VREGD2), U13.15 (VREGD): now also C64.1; no longer C63.1
- net at U13.6 (~{EXTRES}): now also R25.2
- net HIG_CS: no longer names the net of U12.G11 (PG8)
- net VBAT: no longer names the net of J2.1 (Pin_1)
- net VBAT: now also Q1.3
- new net: R37.2, R38.1, U3.3 (CP2)
- new net: C60.1, U3.11 (SS)
- new net: Q3.2 (G1), R45.1
- new net: L1.1, PS1.7 (SW)
- new net: D15.2 (A), R53.2
- new net: PS1.8 (PG), R26.2
- new net: Q3.4 (G2), R51.1
- new net: Q2.3 (S2), Q3.5 (D2), Q3.6 (D2)
- new net: Q2.1 (S1), Q3.7 (D1), Q3.8 (D1)
- new net: Q2.4 (G2), R50.1
- new net: R35.1, U3.10 (ILIM)
- new net: Q1.1, R40.1
- new net: R21.1, U9.B5 (CC2)
- new net: R29.2, R30.1, U3.4 (OV2)
- new net: R27.1, R28.2, U3.6 (PR1)
- new net: Q2.2 (G1), R44.1
- new net: D13.2 (A), R46.2
- new net: C49.1, R39.2
- new net: R20.1, U9.A5 (CC1)
- no-connect marks 31 -> 107
